File: ECE 558/Project3 Hardware/Project3.brd (EAGLE design)
At the start: 58.4 x 32.7 mm, 15 parts, among them IC1 PIC16F676P, IC2 LM35CZ, J1 RASPBERRYPI-40-PIN-GPIO_PTH_N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, M1 MOTOR10MM, T1 2N3904

Commit message: fixed board
Parts:
- removed D1, D2: CLEAR, SparkFun-LED:LED-RGB-THRU
- removed R1, R2: (no value), rcl:0204V
- added U$1, U$2: 5MMRGBLED, led_rgb:LED5MMRGB
- moved R5 13.0 mm to (21.6, 36.7), turned to 90 degrees
- moved M1 11.3 mm to (46.1, 41.9), turned to 0 degrees
- moved D3 5.99 mm to (37.2, 33.8)
- moved R6 4.62 mm to (27.3, 37.5)
Connections:
- removed net N$18: D1.4, R2.2
- removed net N$19: D1.1, R1.2
- net GND: now also U$1.P$3, U$2.P$1, U$2.P$3, U$2.P$4; no longer D1.2, D2.2, R1.1, R2.1
- net N$11: now also U$1.P$4; no longer D2.1
- net N$12: now also U$1.P$2; no longer D2.4
- net N$13: now also R5.2; no longer R6.2
- net N$14: now also R6.1, U$1.P$1; no longer IC1.12, R5.2
- net N$15: now also IC1.12, R6.2; no longer D2.3, R6.1
- net N$17: now also U$2.P$2; no longer D1.3
Routing:
- net N$15: track 26.1 -> 3.96 mm
- net N$2: track 33.9 -> 12.8 mm
- net N$1: track 82.4 -> 65.1 mm
- net N$12: track 4.63 -> 14.7 mm
- net N$14: track 12.0 -> 6.09 mm
- net N$10: track 9.06 -> 4.49 mm
- net N$19: track 4.45 -> 0.00 mm
- net N$18: track 3.81 -> 0.00 mm
- net N$11: track 4.58 -> 6.66 mm
- net N$13: track 4.45 -> 2.67 mm
- net N$17: track 16.7 -> 17.2 mm
- added copper zone on layer 1, net GND
